Commit message: added skid steer plugin

File: urdf/espeleo2.urdf (robot description, URDF)
Before this commit: robot espeleo, 9 links, 8 joints
Links:
- link chassis: mass 0.5 -> 15.0
- link imu_link: mass 0.01 -> 0.05
- link left_back_wheel: mass 0.2 -> 0.8
- link left_front_wheel: mass 0.2 -> 0.8
- link os1_sensor: mass 0.01 -> 0.5
- link right_back_wheel: mass 0.2 -> 0.8
- link right_front_wheel: mass 0.2 -> 0.8
Joints:
- joint left_back_wheel_joint: limit lower=-9.42 upper=9.42 effort=80 velocity=15 -> (none); type revolute -> continuous
- joint left_front_wheel_joint: limit lower=-9.42 upper=9.42 effort=80 velocity=15 -> (none); type revolute -> continuous
- joint right_back_wheel_joint: limit lower=-9.42 upper=9.42 effort=80 velocity=15 -> (none); origin xyz=-0.212 -0.175 -0.01 rpy=3.1415 0 0 -> xyz=-0.212 -0.175 -0.01 rpy=0 0 0; type revolute -> continuous
- joint right_front_wheel_joint: limit lower=-9.42 upper=9.42 effort=80 velocity=15 -> (none); origin xyz=0.215 -0.175 -0.01 rpy=3.1415 0 0 -> xyz=0.215 -0.175 -0.01 rpy=0 0 0; type revolute -> continuous

Commit message: Fix skid steer plugin parameter

File: urdf/espeleo2.urdf (robot description, URDF)
Before this commit: robot espeleo, 9 links, 8 joints
Links:
- link chassis: mass 15.0 -> 20.0

Commit message: Added cameras/hokuyo/imu sensors

File: urdf/espeleo2.urdf (robot description, URDF)
Before this commit: robot espeleo, 9 links, 8 joints
Links:
- added link back_camera, mass 0.05
- added link front_camera, mass 0.05
- added link hokuyo, mass 0.5; collision box size=0.13 0.13 0.095; visual box size=0.01 0.01 0.01
Joints:
- added joint camera2_joint: type fixed, parent chassis, child back_camera, origin xyz=-0.265 0 0.03 rpy=0 0 3.14, axis 0 1 0
- added joint camera_joint: type fixed, parent chassis, child front_camera, origin xyz=0.265 0 0.03 rpy=0 0 0, axis 0 1 0
- added joint laser2_joint: type fixed, parent sensor_tower, child hokuyo, origin xyz=0 0 .305 rpy=0 0 0, axis 0 0 0

Commit message: added velodyne and cameradepth plugins

File: urdf/espeleo2.urdf (robot description, URDF)
Before this commit: robot espeleo, 12 links, 11 joints
Links:
- removed link os1_sensor
- added link d435i_pt_link, mass 0.01
- added link d435i_sim_link, mass 0.01; visual mesh filename=package://espeleo_gazebo/urdf/stl/realsense_d435.STL scale=0.001 0.001 0.001
- added link velodyne, mass 0.01
- added link velodyne_base_link, mass 0.83; collision box size=0.13 0.13 0.095; visual mesh filename=package://espeleo_gazebo/urdf/stl/Lidar.STL scale=0.001 0.001 0.001
- link hokuyo: geometry collision box size=0.01 0.01 0.01; visual box size=0.01 0.01 0.01
- link left_back_wheel: mass 0.8 -> 0.32
- link left_front_wheel: mass 0.8 -> 0.32
- link right_back_wheel: mass 0.8 -> 0.32
- link right_front_wheel: mass 0.8 -> 0.32
Joints:
- removed joint laser_joint
- added joint realsense_d435_pt_joint: type fixed, parent d435i_sim_link, child d435i_pt_link, origin xyz=0 0 0 rpy=-1.57 0 -1.57, axis 0 0 0
- added joint realsense_d435_sim_joint: type fixed, parent sensor_tower, child d435i_sim_link, origin xyz=0.06 0 0.18 rpy=0 0 0, axis 0 0 0
- added joint velodyne_base_mount_joint: type fixed, parent sensor_tower, child velodyne_base_link, origin xyz=0 0 .205 rpy=0 0 0, axis 0 0 0
- added joint velodyne_base_scan_joint: type fixed, parent velodyne_base_link, child velodyne, origin xyz=0 0 0.0377 rpy=0 0 0
